Commit message: add ui for selecting robot, maybe a little bit slow

File: Assets/URDF/mycobot/mycobot_280_m5/mycobot.urdf.xacro (robot description, xacro)
@@ -10,5 +10,5 @@
     <visual>
       <geometry>
-       <mesh filename="package://mycobot_description/urdf/mycobot/mesh/link1.dae"/>
+       <mesh filename="meshes/link1.dae"/>
       </geometry>
       <origin xyz = "0.0 0 0 " rpy = " 0 0 -${pi/2}"/>
@@ -16,5 +16,5 @@
     <collision>
       <geometry>
-       <mesh filename="package://mycobot_description/urdf/mycobot/mesh/link1.dae"/>
+       <mesh filename="meshes/link1.dae"/>
         </geometry>
         <origin xyz = "0.0 0 0 " rpy = " 0 0 -${pi/2}"/>
@@ -29,5 +29,5 @@
     <visual>
       <geometry>
-       <mesh filename="package://mycobot_description/urdf/mycobot/mesh/link2.dae"/>
+       <mesh filename="meshes/link2.dae"/>
       </geometry>
       <origin xyz = "0.0 0 -0.06096 " rpy = " 0 0 -${pi/2}"/>
@@ -35,5 +35,5 @@
     <collision>
      <geometry>
-       <mesh filename="package://mycobot_description/urdf/mycobot/mesh/link2.dae"/>
+       <mesh filename="meshes/link2.dae"/>
       </geometry>
       <origin xyz = "0.0 0 -0.06096 " rpy = " 0 0 -${pi/2}"/>
@@ -48,5 +48,5 @@
     <visual>
       <geometry>
-       <mesh filename="package://mycobot_description/urdf/mycobot/mesh/link3.dae"/>
+       <mesh filename="meshes/link3.dae"/>
       </geometry>
     <origin xyz = "0.0 0 0.03256 " rpy = " 0 -${pi/2} 0"/>
@@ -54,5 +54,5 @@
     <collision>
       <geometry>
-       <mesh filename="package://mycobot_description/urdf/mycobot/mesh/link3.dae"/>
+       <mesh filename="meshes/link3.dae"/>
       </geometry>
       <origin xyz = "0.0 0 0.03256 " rpy = " 0 -${pi/2} 0"/>
@@ -68,5 +68,5 @@
       <geometry>
        <!--- 0.0 0 -0.04 -->
-       <mesh filename="package://mycobot_description/urdf/mycobot/mesh/link4.dae"/>
+       <mesh filename="meshes/link4.dae"/>
       </geometry>
       <origin xyz = "0.0 0 0.03056 " rpy = " 0 -${pi/2} 0"/>
@@ -75,5 +75,5 @@
       <geometry>
        <!--- 0.0 0 -0.04 -->
-       <mesh filename="package://mycobot_description/urdf/mycobot/mesh/link4.dae"/>
+       <mesh filename="meshes/link4.dae"/>
       </geometry>
       <origin xyz = "0.0 0 0.03056 " rpy = " 0 -${pi/2} 0"/>
@@ -89,5 +89,5 @@
       <geometry>
        <!--- 0.0 0 -0.04 -->
-       <mesh filename="package://mycobot_description/urdf/mycobot/mesh/link5.dae"/>
+       <mesh filename="meshes/link5.dae"/>
       </geometry>
     <origin xyz = "0.0 0 -0.03356 " rpy = " -${pi/2} 0 0"/>
@@ -96,5 +96,5 @@
        <geometry>
        <!--- 0.0 0 -0.04 -->
-       <mesh filename="package://mycobot_description/urdf/mycobot/mesh/link5.dae"/>
+       <mesh filename="meshes/link5.dae"/>
       </geometry>
       <origin xyz = "0.0 0 -0.03356 " rpy = " -${pi/2} 0 0"/>
@@ -110,5 +110,5 @@
       <geometry>
        <!--- 0.0 0 -0.04 -->
-       <mesh filename="package://mycobot_description/urdf/mycobot/mesh/link6.dae"/>
+       <mesh filename="meshes/link6.dae"/>
       </geometry>
     <origin xyz = "0 0.00 -0.038 " rpy = " 0 0 0"/>
@@ -117,5 +117,5 @@
       <geometry>
        <!--- 0.0 0 -0.04 -->
-       <mesh filename="package://mycobot_description/urdf/mycobot/mesh/link6.dae"/>
+       <mesh filename="meshes/link6.dae"/>
       </geometry>
     <origin xyz = "0 0.00 -0.038 " rpy = " 0 0 0"/>
@@ -131,5 +131,5 @@
       <geometry>
        <!--- 0.0 0 -0.04 -->
-       <mesh filename="package://mycobot_description/urdf/mycobot/mesh/link7.dae"/>
+       <mesh filename="meshes/link7.dae"/>
       </geometry>
     <origin xyz = "0.0 0 -0.012 " rpy = " 0 0 0"/>
@@ -138,5 +138,5 @@
       <geometry>
        <!--- 0.0 0 -0.04 -->
-       <mesh filename="package://mycobot_description/urdf/mycobot/mesh/link7.dae"/>
+       <mesh filename="meshes/link7.dae"/>
       </geometry>
     <origin xyz = "0.0 0 -0.012 " rpy = " 0 0 0"/>
